Commit message: update rotorx atom urdf

File: rotors_description/urdf/atom.xacro (robot description, xacro)
@@ -19,18 +19,21 @@
   <xacro:property name="namespace" value="$(arg namespace)" />
   <xacro:property name="rotor_velocity_slowdown_sim" value="10" />
-  <xacro:property name="use_mesh_file" value="true" />
-  <xacro:property name="mesh_file" value="package://rotors_description/meshes/hummingbird.dae" />
-  <xacro:property name="mass" value="0.68" /> <!-- [kg] -->
+  <xacro:property name="use_mesh_file" value="false" />
+  <xacro:property name="mesh_file" value="package://rotors_description/meshes/atom.stl" />
+  <xacro:property name="mass" value="0.164" /> <!-- [kg] -->
   <xacro:property name="body_width" value="0.1" /> <!-- [m] -->
-  <xacro:property name="body_height" value="0.12" /> <!-- [m] -->
+  <xacro:property name="body_height" value="0.08" /> <!-- [m] -->
   <xacro:property name="mass_rotor" value="0.009" /> <!-- [kg] -->
-  <xacro:property name="arm_length" value="0.17" /> <!-- [m] -->
+  <xacro:property name="front_arm_x" value="0.03" /> <!-- [m] -->
+  <xacro:property name="front_arm_y" value="0.065" /> <!-- [m] -->
+  <xacro:property name="back_arm_x" value="0.05" /> <!-- [m] -->
+  <xacro:property name="back_arm_y" value="0.05" /> <!-- [m] -->
   <xacro:property name="rotor_offset_top" value="0.01" /> <!-- [m] -->
-  <xacro:property name="radius_rotor" value="0.1" /> <!-- [m] -->
+  <xacro:property name="radius_rotor" value="0.037" /> <!-- [m] -->
   <xacro:property name="motor_constant" value="8.54858e-06" /> <!-- [kg m/s^2] -->
   <xacro:property name="moment_constant" value="0.016" /> <!-- [m] -->
   <xacro:property name="time_constant_up" value="0.0125" /> <!-- [s] -->
   <xacro:property name="time_constant_down" value="0.025" /> <!-- [s] -->
-  <xacro:property name="max_rot_velocity" value="838" /> <!-- [rad/s] -->
+  <xacro:property name="max_rot_velocity" value="6000" /> <!-- [rad/s] -->
   <xacro:property name="rotor_drag_coefficient" value="8.06428e-05" />
   <xacro:property name="rolling_moment_coefficient" value="0.000001" />
@@ -41,5 +44,5 @@
   <!-- inertia of a single rotor, assuming it is a cuboid. Height=3mm, width=15mm -->
   <xacro:property name="rotor_inertia">
-    <xacro:box_inertia x="${radius_rotor}" y="0.015" z="0.003" mass="${mass_rotor*rotor_velocity_slowdown_sim}" />
+    <xacro:box_inertia x="${radius_rotor}" y="0.003" z="0.003" mass="${mass_rotor*rotor_velocity_slowdown_sim}" />
   </xacro:property>
   <!-- Included URDF Files -->
@@ -58,6 +61,6 @@
   <xacro:vertical_rotor
     robot_namespace="${namespace}"
-    suffix="front"
-    direction="cw"
+    suffix="front_right"
+    direction="ccw"
     motor_constant="${motor_constant}"
     moment_constant="${moment_constant}"
@@ -74,10 +77,52 @@
     use_own_mesh="false"
     mesh="">
-    <origin xyz="${arm_length} 0 ${rotor_offset_top}" rpy="0 0 0" />
+    <origin xyz="${front_arm_x} -${front_arm_y} ${rotor_offset_top}" rpy="0 0 0" />
     <xacro:insert_block name="rotor_inertia" />
   </xacro:vertical_rotor>
   <xacro:vertical_rotor
     robot_namespace="${namespace}"
-    suffix="left"
+    suffix="front_left"
+    direction="cw"
+    motor_constant="${motor_constant}"
+    moment_constant="${moment_constant}"
+    parent="${namespace}/base_link"
+    mass_rotor="${mass_rotor}"
+    radius_rotor="${radius_rotor}"
+    time_constant_up="${time_constant_up}"
+    time_constant_down="${time_constant_down}"
+    max_rot_velocity="${max_rot_velocity}"
+    motor_number="2"
+    rotor_drag_coefficient="${rotor_drag_coefficient}"
+    rolling_moment_coefficient="${rolling_moment_coefficient}"
+    color="Blue"
+    use_own_mesh="false"
+    mesh="">
+    <origin xyz="${front_arm_x} ${front_arm_y} ${rotor_offset_top}" rpy="0 0 0" />
+    <xacro:insert_block name="rotor_inertia" />
+  </xacro:vertical_rotor>
+  <xacro:vertical_rotor
+    robot_namespace="${namespace}"
+    suffix="back"
+    direction="cw"
+    motor_constant="${motor_constant}"
+    moment_constant="${moment_constant}"
+    parent="${namespace}/base_link"
+    mass_rotor="${mass_rotor}"
+    radius_rotor="${radius_rotor}"
+    time_constant_up="${time_constant_up}"
+    time_constant_down="${time_constant_down}"
+    max_rot_velocity="${max_rot_velocity}"
+    motor_number="3"
+    rotor_drag_coefficient="${rotor_drag_coefficient}"
+    rolling_moment_coefficient="${rolling_moment_coefficient}"
+    color="Blue"
+    use_own_mesh="false"
+    mesh="">
+    <origin xyz="-${back_arm_x} -${back_arm_y} ${rotor_offset_top}" rpy="0 0 0" />
+    <xacro:insert_block name="rotor_inertia" />
+  </xacro:vertical_rotor>
+  <xacro:vertical_rotor
+    robot_namespace="${namespace}"
+    suffix="right"
     direction="ccw"
     motor_constant="${motor_constant}"
@@ -95,47 +140,5 @@
     use_own_mesh="false"
     mesh="">
-    <origin xyz="0 ${arm_length} ${rotor_offset_top}" rpy="0 0 0" />
-    <xacro:insert_block name="rotor_inertia" />
-  </xacro:vertical_rotor>
-  <xacro:vertical_rotor
-    robot_namespace="${namespace}"
-    suffix="back"
-    direction="cw"
-    motor_constant="${motor_constant}"
-    moment_constant="${moment_constant}"
-    parent="${namespace}/base_link"
-    mass_rotor="${mass_rotor}"
-    radius_rotor="${radius_rotor}"
-    time_constant_up="${time_constant_up}"
-    time_constant_down="${time_constant_down}"
-    max_rot_velocity="${max_rot_velocity}"
-    motor_number="2"
-    rotor_drag_coefficient="${rotor_drag_coefficient}"
-    rolling_moment_coefficient="${rolling_moment_coefficient}"
-    color="Blue"
-    use_own_mesh="false"
-    mesh="">
-    <origin xyz="-${arm_length} 0 ${rotor_offset_top}" rpy="0 0 0" />
-    <xacro:insert_block name="rotor_inertia" />
-  </xacro:vertical_rotor>
-  <xacro:vertical_rotor
-    robot_namespace="${namespace}"
-    suffix="right"
-    direction="ccw"
-    motor_constant="${motor_constant}"
-    moment_constant="${moment_constant}"
-    parent="${namespace}/base_link"
-    mass_rotor="${mass_rotor}"
-    radius_rotor="${radius_rotor}"
-    time_constant_up="${time_constant_up}"
-    time_constant_down="${time_constant_down}"
-    max_rot_velocity="${max_rot_velocity}"
-    motor_number="3"
-    rotor_drag_coefficient="${rotor_drag_coefficient}"
-    rolling_moment_coefficient="${rolling_moment_coefficient}"
-    color="Blue"
-    use_own_mesh="false"
-    mesh="">
-    <origin xyz="0 -${arm_length} ${rotor_offset_top}" rpy="0 0 0" />
+    <origin xyz="-${back_arm_x} ${back_arm_y} ${rotor_offset_top}" rpy="0 0 0" />
     <xacro:insert_block name="rotor_inertia" />
   </xacro:vertical_rotor>

Commit message: Mat's updated rotorx atom model

File: rotors_description/urdf/atom.xacro (robot description, xacro)
@@ -22,11 +22,11 @@
   <xacro:property name="mesh_file" value="package://rotors_description/meshes/atom.stl" />
   <xacro:property name="mass" value="0.164" /> <!-- [kg] -->
-  <xacro:property name="body_width" value="0.1" /> <!-- [m] -->
-  <xacro:property name="body_height" value="0.08" /> <!-- [m] -->
-  <xacro:property name="mass_rotor" value="0.009" /> <!-- [kg] -->
-  <xacro:property name="front_arm_x" value="0.03" /> <!-- [m] -->
-  <xacro:property name="front_arm_y" value="0.065" /> <!-- [m] -->
-  <xacro:property name="back_arm_x" value="0.05" /> <!-- [m] -->
-  <xacro:property name="back_arm_y" value="0.05" /> <!-- [m] -->
+  <xacro:property name="body_width" value="0.09" /> <!-- [m] -->
+  <xacro:property name="body_height" value="0.07" /> <!-- [m] -->
+  <xacro:property name="mass_rotor" value="0.0005" /> <!-- [kg] -->
+  <xacro:property name="front_arm_x" value="0.029" /> <!-- [m] -->
+  <xacro:property name="front_arm_y" value="0.055" /> <!-- [m] -->
+  <xacro:property name="back_arm_x" value="0.045" /> <!-- [m] -->
+  <xacro:property name="back_arm_y" value="0.040" /> <!-- [m] -->
   <xacro:property name="rotor_offset_top" value="0.01" /> <!-- [m] -->
   <xacro:property name="radius_rotor" value="0.037" /> <!-- [m] -->
@@ -40,9 +40,9 @@
   <!-- Property Blocks -->
   <xacro:property name="body_inertia">
-    <inertia ixx="0.007" ixy="0.0" ixz="0.0" iyy="0.007" iyz="0.0" izz="0.012" /> <!-- [kg m^2] [kg m^2] [kg m^2] [kg m^2] [kg m^2] [kg m^2] -->
+    <inertia ixx="0.000145" ixy="0.0" ixz="0.0" iyy="0.000106" iyz="0.0" izz="0.000199" /> <!-- [kg m^2] [kg m^2] [kg m^2] [kg m^2] [kg m^2] [kg m^2] -->
   </xacro:property>
   <!-- inertia of a single rotor, assuming it is a cuboid. Height=3mm, width=15mm -->
   <xacro:property name="rotor_inertia">
-    <xacro:box_inertia x="${radius_rotor}" y="0.003" z="0.003" mass="${mass_rotor*rotor_velocity_slowdown_sim}" />
+    <xacro:box_inertia x="${radius_rotor}" y="0.005" z="0.003" mass="${mass_rotor*rotor_velocity_slowdown_sim}" />
   </xacro:property>
   <!-- Included URDF Files -->
