Commit message: Add generic wrench subscriber for buoyancy

File: rotors_description/urdf/blimp.xacro (robot description, xacro)
@@ -57,4 +57,32 @@
     <xacro:insert_block name="body_inertia" />
   </xacro:multirotor_base_macro>
+  <joint name="${namespace}/buoyancy_joint" type="fixed">
+    <origin xyz="0 0 0.75" rpy="0 0 0" />
+    <parent link="${namespace}/base_link" />
+    <child link="${namespace}/buoyancy_visual" />
+  </joint>
+  <link name="${namespace}/buoyancy_visual">
+    <visual>
+      <origin xyz="0 0 0" rpy="0 0 0" />
+      <geometry>
+	<sphere radius="0.51"/>
+      </geometry>
+    </visual>
+    <collision>
+      <origin xyz="0 0 0" rpy="0 0 0" />
+      <geometry>
+	<sphere radius="0.51"/>
+      </geometry>
+    </collision>
+  </link>
+  <gazebo>
+    <plugin name="buoyancy_force" filename="libgazebo_ros_force.so">
+      <alwaysOn>true</alwaysOn>
+      <update>100</update>
+      <updateRate>100.0</updateRate>
+      <bodyName>${namespace}/buoyancy_visual</bodyName>
+      <topicName>buoyant_wrench</topicName>
+    </plugin>
+  </gazebo>
   <!-- Instantiate rotors -->
   <xacro:vertical_rotor

Commit message: Fix blimp urdf

File: rotors_description/urdf/blimp.xacro (robot description, xacro)
@@ -39,5 +39,5 @@
   <!-- Property Blocks -->
   <xacro:property name="body_inertia">
-    <inertia ixx="0.007" ixy="0.0" ixz="0.0" iyy="0.007" iyz="0.0" izz="0.012" /> <!-- [kg m^2] [kg m^2] [kg m^2] [kg m^2] [kg m^2] [kg m^2] -->
+    <inertia ixx="0.6" ixy="0.0" ixz="0.0" iyy="0.6" iyz="0.0" izz="0.6" /> <!-- [kg m^2] [kg m^2] [kg m^2] [kg m^2] [kg m^2] [kg m^2] -->
   </xacro:property>
   <!-- inertia of a single rotor, assuming it is a cuboid. Height=3mm, width=15mm -->
@@ -171,7 +171,7 @@
   </xacro:vertical_rotor>
   <!-- Instantiate thrusters -->
-  <xacro:axis_rotor
-    robot_namespace="${namespace}"
-    suffix="x_thrust"
+  <xacro:vertical_rotor
+    robot_namespace="${namespace}"
+    suffix="x_thrust_cw"
     direction="cw"
     motor_constant="${motor_constant}"
@@ -189,12 +189,11 @@
     use_own_mesh="false"
     mesh="">
-    <axis xyz="1 0 0" />
-    <origin xyz="${arm_length} 0 0" rpy="0 0 0" />
-    <xacro:insert_block name="rotor_inertia" />
-  </xacro:axis_rotor>
-  <xacro:axis_rotor
-    robot_namespace="${namespace}"
-    suffix="y_thrust"
-    direction="cw"
+    <origin xyz="${arm_length} ${arm_length/2} 0" rpy="0 ${pi/2} 0" />
+    <xacro:insert_block name="rotor_inertia" />
+  </xacro:vertical_rotor>
+  <xacro:vertical_rotor
+    robot_namespace="${namespace}"
+    suffix="x_thrust_ccw"
+    direction="ccw"
     motor_constant="${motor_constant}"
     moment_constant="${moment_constant}"
@@ -211,7 +210,48 @@
     use_own_mesh="false"
     mesh="">
-    <axis xyz="0 1 0" />
-    <origin xyz="0 ${arm_length} 0" rpy="0 0 0" />
-    <xacro:insert_block name="rotor_inertia" />
-  </xacro:axis_rotor>
+    <origin xyz="${arm_length} ${-arm_length/2} 0" rpy="0 ${pi/2} 0" />
+    <xacro:insert_block name="rotor_inertia" />
+  </xacro:vertical_rotor>
+  <xacro:vertical_rotor
+    robot_namespace="${namespace}"
+    suffix="y_thrust_cw"
+    direction="cw"
+    motor_constant="${motor_constant}"
+    moment_constant="${moment_constant}"
+    parent="${namespace}/base_link"
+    mass_rotor="${mass_rotor}"
+    radius_rotor="${radius_rotor}"
+    time_constant_up="${time_constant_up}"
+    time_constant_down="${time_constant_down}"
+    max_rot_velocity="${max_rot_velocity}"
+    motor_number="6"
+    rotor_drag_coefficient="${rotor_drag_coefficient}"
+    rolling_moment_coefficient="${rolling_moment_coefficient}"
+    color="Black"
+    use_own_mesh="false"
+    mesh="">
+    <origin xyz="${arm_length/2} ${arm_length} 0" rpy="${-pi/2} 0 0" />
+    <xacro:insert_block name="rotor_inertia" />
+  </xacro:vertical_rotor>
+  <xacro:vertical_rotor
+    robot_namespace="${namespace}"
+    suffix="y_thrust_ccw"
+    direction="ccw"
+    motor_constant="${motor_constant}"
+    moment_constant="${moment_constant}"
+    parent="${namespace}/base_link"
+    mass_rotor="${mass_rotor}"
+    radius_rotor="${radius_rotor}"
+    time_constant_up="${time_constant_up}"
+    time_constant_down="${time_constant_down}"
+    max_rot_velocity="${max_rot_velocity}"
+    motor_number="7"
+    rotor_drag_coefficient="${rotor_drag_coefficient}"
+    rolling_moment_coefficient="${rolling_moment_coefficient}"
+    color="Black"
+    use_own_mesh="false"
+    mesh="">
+    <origin xyz="${-arm_length/2} ${arm_length} 0" rpy="${-pi/2} 0 0" />
+    <xacro:insert_block name="rotor_inertia" />
+  </xacro:vertical_rotor>
 </robot>

File: rotors_description/urdf/multirotor_base.xacro (robot description, xacro)
@@ -74,9 +74,9 @@
   </xacro:macro>
   <!-- Rotor joint and link -->
-  <xacro:macro name="axis_rotor"
-    params="robot_namespace suffix direction motor_constant moment_constant parent mass_rotor radius_rotor time_constant_up time_constant_down max_rot_velocity motor_number rotor_drag_coefficient rolling_moment_coefficient color use_own_mesh mesh *axis *origin *inertia">
+  <xacro:macro name="vertical_rotor"
+    params="robot_namespace suffix direction motor_constant moment_constant parent mass_rotor radius_rotor time_constant_up time_constant_down max_rot_velocity motor_number rotor_drag_coefficient rolling_moment_coefficient color use_own_mesh mesh *origin *inertia">
     <joint name="${robot_namespace}/rotor_${motor_number}_joint" type="continuous">
       <xacro:insert_block name="origin" />
-      <xacro:insert_block name="axis" />
+      <axis xyz="0 0 1" />
       <!-- TODO(ff): not currently set because it's not yet supported -->
       <!-- <limit effort="2000" velocity="${max_rot_velocity}" /> -->
@@ -132,28 +132,3 @@
     </gazebo>
   </xacro:macro>
-  <xacro:macro name="vertical_rotor"
-	       params="robot_namespace suffix direction motor_constant moment_constant parent mass_rotor radius_rotor time_constant_up time_constant_down max_rot_velocity motor_number rotor_drag_coefficient rolling_moment_coefficient color use_own_mesh mesh *origin *inertia">
-    <xacro:axis_rotor
-      robot_namespace="${robot_namespace}"
-      suffix="${suffix}"
-      direction="${direction}"
-      motor_constant="${motor_constant}"
-      moment_constant="${moment_constant}"
-      parent="${parent}"
-      mass_rotor="${mass_rotor}"
-      radius_rotor="${radius_rotor}"
-      time_constant_up="${time_constant_up}"
-      time_constant_down="${time_constant_down}"
-      max_rot_velocity="${max_rot_velocity}"
-      motor_number="${motor_number}"
-      rotor_drag_coefficient="${rotor_drag_coefficient}"
-      rolling_moment_coefficient="${rolling_moment_coefficient}"
-      color="${color}"
-      use_own_mesh="${use_own_mesh}"
-      mesh="${mesh}">
-      <axis xyz="0 0 1" />
-      <xacro:insert_block name="origin" />
-      <xacro:insert_block name="rotor_inertia" />
-    </xacro:axis_rotor>
-  </xacro:macro>
 </robot>
